File: hardware/pcb/octessera.kicad_sch (KiCad schematic)
At the start: 11 parts, among them J1 NeoTrellis_Conn, SW1 RotaryEncoder_Switch, SW2 RotaryEncoder_Switch, SW3 RotaryEncoder_Switch, SW4 RotaryEncoder_Switch, U1 Raspberry Zero 2 W, U2 SSD1351, U3 USB-C, U4 PCM5102a, U5 NeoKey

Commit message: Update PCB protection and fabrication outputs
Parts:
- added D1: SA5.0A, Diode_THT:D_DO-15_P10.16mm_Horizontal, symbol Device:D_Zener
Connections:
- net +5V: now also D1.1 (K)
- net GND: now also D1.2 (A)
- no-connect marks 0 -> 20
Other:
- moved on the sheet: U3
